File: Storage_Armature_MCU_PCB.kicad_sch (KiCad schematic)
At the start: 117 parts, among them J2 ERROR, Q1 20N06, Q2 20N06, U14 USBLC6-2P6, U22 LTV-247, U4 ADP3338AKCZ-3.3RL7, U5 ADP3338AKCZ-3.3RL7

Commit message: VER1.0: добавил светодиоды аварии и гребенку для анализатора
Parts:
- added D24, D25, D26: (no value), LED_SMD:LED_1206_3216Metric_Pad1.42x1.75mm_HandSolder, symbol Device:LED_Small
- added J3: User, Connector_PinSocket_2.54mm:PinSocket_2x08_P2.54mm_Vertical, symbol Connector_Generic:Conn_02x08_Odd_Even
Connections:
- net ERROR_LvL1_IN: now also D24.2 (A); no longer R92.1
- net ERROR_LvL2_IN: now also D25.2 (A); no longer R94.1
- net ERROR_LvL3_IN: now also D26.2 (A); no longer R95.1
- net GND: now also J3.10 (Pin_10), J3.12 (Pin_12), J3.14 (Pin_14), J3.16 (Pin_16), J3.2 (Pin_2), J3.4 (Pin_4), J3.6 (Pin_6), J3.8 (Pin_8)
- net GPIO1: now reaches U1.33 (PB12)
- net GPIO1: now also J3.1 (Pin_1)
- net GPIO2: now reaches U1.34 (PB13)
- net GPIO2: now also J3.3 (Pin_3)
- net GPIO3: now reaches U1.35 (PB14)
- net GPIO3: now also J3.5 (Pin_5)
- net GPIO4: now reaches U1.36 (PB15)
- net GPIO4: now also J3.7 (Pin_7)
- net GPIO5: now reaches U1.37 (PC6)
- net GPIO5: now also J3.9 (Pin_9)
- net GPIO6: now reaches U1.38 (PC7)
- net GPIO6: now also J3.11 (Pin_11)
- net GPIO7: now reaches U1.39 (PC8)
- net GPIO7: now also J3.13 (Pin_13)
- net GPIO8: now reaches U1.40 (PC9)
- net GPIO8: now also J3.15 (Pin_15)
- new net: D26.1 (K), R95.1
- new net: D25.1 (K), R94.1
- new net: D24.1 (K), R92.1
Other:
- moved on the sheet: J2
