File: Storage_Armature_MCU_PCB.kicad_sch (KiCad schematic)
At the start: 121 parts, among them Y1 16M

Commit message: VER1.0: обновил шелкографию, гербера и BOM
Parts:
- D17, D7: Product Name FYLS-0603UBC -> FYLS-0805UBC
- D24, D25, D26: Product Name FYLS-0603UBC -> FYLS-1206UBC
- J1: Product Name KLS1-207-1-04-S -> DS-1021-1x4; Replacement DS-1021-1x4 -> KLS1-207-1-04-S
- J3: Product Name KLS1-207-2-16-S -> DS1021-2x8; Replacement (none) -> KLS1-207-2-16-S
- R1, R2, R37, R40, R47, R48, R49, R54, R55, R6, R78, R87, R88, R89, R90, R91, R92, R93, R94, R95, R96, R97: Description P/N Resistor SMD -> Resistor SMD 1%
- R39: value 750 -> 1k; Description P/N Resistor SMD -> Resistor SMD 1%
- R57, R58: value 1.1k -> 1k; Description P/N Resistor SMD -> Resistor SMD 1%
- U14: Product Name USBLC6-2P6 -> USBLC6-2SC6
Changed lines of the file:
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@@
 			)
 		)
-		(property "Description P/N" "Resistor SMD"
+		(property "Description P/N" "Resistor SMD 1%"
 			(at 170.18 502.92 0)
 			(hide yes)
@@
 			)
 		)
-		(property "Description P/N" "Resistor SMD"
+		(property "Description P/N" "Resistor SMD 1%"
 			(at 612.14 309.88 0)
 			(hide yes)
@@
 			)
 		)
-		(property "Product Name" "USBLC6-2P6"
+		(property "Product Name" "USBLC6-2SC6"
 			(at 626.11 302.26 0)
 			(hide yes)
@@
 			)
 		)
-		(property "Product Name" "FYLS-0603UBC"
+		(property "Product Name" "FYLS-0805UBC"
 			(at 529.59 335.28 0)
 			(hide yes)
@@
 			)
 		)
-		(property "Replacement" "DS-1021-1x4"
+		(property "Replacement" "KLS1-207-1-04-S"
 			(at 650.24 302.26 0)
 			(hide yes)
@@
 			)
 		)
-		(property "Product Name" "KLS1-207-1-04-S"
+		(property "Product Name" "DS-1021-1x4 "
 			(at 650.24 302.26 0)
 			(hide yes)
@@
 			)
 		)
-		(property "Description P/N" "Resistor SMD"
+		(property "Description P/N" "Resistor SMD 1%"
 			(at 137.16 505.46 90)
 			(hide yes)
@@
 			)
 		)
-		(property "Description P/N" "Resistor SMD"
+		(property "Description P/N" "Resistor SMD 1%"
 			(at 365.76 424.18 90)
 			(hide yes)
@@
 			)
 		)
-		(property "Value" "1.1k"
+		(property "Value" "1k"
 			(at 158.115 245.11 0)
 			(show_name no)
@@
 			)
 		)
-		(property "Description P/N" "Resistor SMD"
+		(property "Description P/N" "Resistor SMD 1%"
 			(at 156.845 246.38 0)
 			(hide yes)
@@
 			)
 		)
-		(property "Product Name" "FYLS-0603UBC"
+		(property "Product Name" "FYLS-1206UBC"
 			(at 124.46 486.41 0)
 			(hide yes)
@@
 			)
 		)
-		(property "Description P/N" "Resistor SMD"
+		(property "Description P/N" "Resistor SMD 1%"
 			(at 161.29 195.58 0)
 			(hide yes)
@@
 			)
 		)
-		(property "Description P/N" "Resistor SMD"
+		(property "Description P/N" "Resistor SMD 1%"
 			(at 280.67 204.47 0)
 			(hide yes)
@@
 			)
 		)
-		(property "Description P/N" "Resistor SMD"
+		(property "Description P/N" "Resistor SMD 1%"
 			(at 137.16 467.36 90)
 			(hide yes)
@@
 			)
 		)
-		(property "Description P/N" "Resistor SMD"
+		(property "Description P/N" "Resistor SMD 1%"
 			(at 280.67 199.39 0)
 			(hide yes)
@@
 			)
 		)
-		(property "Description P/N" "Resistor SMD"
+		(property "Description P/N" "Resistor SMD 1%"
 			(at 612.14 327.66 0)
 			(hide yes)
@@
 			)
 		)
-		(property "Description P/N" "Resistor SMD"
+		(property "Description P/N" "Resistor SMD 1%"
 			(at 121.92 196.85 0)
 			(hide yes)
@@
 			)
 		)
-		(property "Product Name" "FYLS-0603UBC"
+		(property "Product Name" "FYLS-1206UBC"
 			(at 124.46 467.36 0)
 			(hide yes)
@@
 			)
 		)
-		(property "Value" "1.1k"
+		(property "Value" "1k"
 			(at 165.1 302.26 0)
 			(show_name no)
@@
 			)
 		)
-		(property "Description P/N" "Resistor SMD"
+		(property "Description P/N" "Resistor SMD 1%"
 			(at 163.83 303.53 0)
 			(hide yes)
@@
 			)
 		)
-		(property "Product Name" "FYLS-0603UBC"
+		(property "Product Name" "FYLS-0805UBC"
 			(at 538.48 335.28 0)
 			(hide yes)
@@
 			)
 		)
-		(property "Product Name" "FYLS-0603UBC"
+		(property "Product Name" "FYLS-1206UBC"
 			(at 124.46 505.46 0)
 			(hide yes)
@@
 			)
 		)
-		(property "Description P/N" "Resistor SMD"
+		(property "Description P/N" "Resistor SMD 1%"
 			(at 160.02 464.82 0)
 			(hide yes)
@@
 			)
 		)
-		(property "Description P/N" "Resistor SMD"
+		(property "Description P/N" "Resistor SMD 1%"
 			(at 137.16 486.41 90)
 			(hide yes)
@@
 			)
 		)
-		(property "Description P/N" "Resistor SMD"
+		(property "Description P/N" "Resistor SMD 1%"
 			(at 529.59 261.62 0)
 			(hide yes)
@@
 			)
 		)
-		(property "Description P/N" "Resistor SMD"
+		(property "Description P/N" "Resistor SMD 1%"
 			(at 165.1 483.87 0)
 			(hide yes)
@@
 			)
 		)
-		(property "Description P/N" "Resistor SMD"
+		(property "Description P/N" "Resistor SMD 1%"
 			(at 538.48 340.36 0)
 			(hide yes)
@@
 			)
 		)
-		(property "Description P/N" "Resistor SMD"
+		(property "Description P/N" "Resistor SMD 1%"
 			(at 551.18 261.62 0)
 			(hide yes)
@@
 			)
 		)
-		(property "Product Name" "KLS1-207-2-16-S"
+		(property "Product Name" "DS1021-2x8 "
 			(at 643.89 346.71 0)
 			(hide yes)
@@
 			)
 		)
-		(property "Replacement" ""
+		(property "Replacement" "KLS1-207-2-16-S"
 			(at 643.89 346.71 0)
 			(hide yes)
@@
 			)
 		)
-		(property "Description P/N" "Resistor SMD"
+		(property "Description P/N" "Resistor SMD 1%"
 			(at 283.21 270.51 0)
 			(hide yes)
@@
 			)
 		)
-		(property "Value" "750"
+		(property "Value" "1k"
 			(at 147.955 343.535 0)
 			(show_name no)
@@
 			)
 		)
-		(property "Description P/N" "Resistor SMD"
+		(property "Description P/N" "Resistor SMD 1%"
 			(at 146.685 344.805 0)
 			(hide yes)
@@
 			)
 		)
-		(property "Description P/N" "Resistor SMD"
+		(property "Description P/N" "Resistor SMD 1%"
 			(at 115.57 187.96 0)
 			(hide yes)
@@
 			)
 		)
-		(property "Description P/N" "Resistor SMD"
+		(property "Description P/N" "Resistor SMD 1%"
 			(at 529.59 340.36 0)
 			(hide yes)
@@
 			)
 		)
-		(property "Description P/N" "Resistor SMD"
+		(property "Description P/N" "Resistor SMD 1%"
 			(at 636.27 299.72 0)
 			(hide yes)
@@
 			)
 		)
-		(property "Description P/N" "Resistor SMD"
+		(property "Description P/N" "Resistor SMD 1%"
 			(at 636.27 302.26 0)
 			(hide yes)
@@
 			)
 		)
-		(property "Description P/N" "Resistor SMD"
+		(property "Description P/N" "Resistor SMD 1%"
 			(at 283.21 265.43 0)
 			(hide yes)
