File: Storage_Armature_MCU_PCB.kicad_pcb (KiCad board)
At the start: 4 copper layers, 163 x 221 mm, 382 parts, among them Y1 16M

Commit message: VER1.0: обновил шелкографию, гербера и BOM
Parts:
- removed the G*** at (241.8, 109.2)
- added G***: LOGO, Logo_My:Logo_Company3, F.Cu at (302.8, 152.5)
- R39: value 750 -> 1k
- R57, R58: value 1.1k -> 1k
