File: Sch/Measure.kicad_sch (KiCad schematic)
At the start: 26 parts, among them U2 NSI1200, U6 OPA333

Commit message: VER1.0: добавил BOM и гербера
Parts:
- C10, C16, C17, C18, C19, C22, C23, C3, C4: Description P/N (none) -> Capacitor SMD 50V
- J28: Product Name DS1073-01-2x1-MVT6 -> DS1073-01-2x1MR2T6
- R10, R11, R21, R3, R5, R7, R79, R8, R9: Description P/N (none) -> Resistor SMD
- TP1, TP17, TP25, TP9: now left out of the parts list
- U2: value NSI1200 -> (none); Description P/N (none) -> Digital Isolator; Product Name (none) -> NSI1200
- U6: value OPA333 -> (none); Description P/N (none) -> Op-Amp; Product Name (none) -> OPA333
