File: Sch/Solenoid_control.kicad_sch (KiCad schematic)
At the start: 13 parts, among them U23 RSCD06D3

Commit message: VER1.0: добавил BOM и гербера
Parts:
- C82: Description P/N (none) -> Capacitor SMD 50V
- F1: value MF-SM075/60-2 -> (none); Description P/N (none) -> Fuse SMD; Product Name (none) -> MF-SM075/60-2
- J24: Product Name DS1073-01-2x1-MVT6 -> DS1073-01-2x1MR2T6
- R108, R109, R110, R120: Description P/N (none) -> Resistor SMD
- U23: value RSCD06D3 -> (none); Description P/N (none) -> Relay; Product Name (none) -> RSCD06D3
Changed lines of the file:
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@@
 			)
 		)
-		(property "Value" "RSCD06D3"
+		(property "Value" ""
 			(at 152.4 101.6 0)
 			(show_name no)
@@
 		)
 		(property "Description" ""
+			(at 152.4 96.52 0)
+			(hide yes)
+			(show_name no)
+			(do_not_autoplace no)
+			(effects
+				(font
+					(size 1.27 1.27)
+				)
+			)
+		)
+		(property "Product Name" "RSCD06D3"
+			(at 152.4 96.52 0)
+			(hide yes)
+			(show_name no)
+			(do_not_autoplace no)
+			(effects
+				(font
+					(size 1.27 1.27)
+				)
+			)
+		)
+		(property "Description P/N" "Relay"
 			(at 152.4 96.52 0)
 			(hide yes)
@@
 			)
 		)
-		(property "Description P/N" ""
+		(property "Description P/N" "Resistor SMD"
 			(at 166.37 106.68 0)
 			(hide yes)
@@
 			)
 		)
-		(property "Description P/N" ""
+		(property "Description P/N" "Resistor SMD"
 			(at 137.16 96.52 0)
 			(hide yes)
@@
 			)
 		)
-		(property "Description P/N" ""
+		(property "Description P/N" "Resistor SMD"
 			(at 124.46 105.41 0)
 			(hide yes)
@@
 			)
 		)
-		(property "Product Name" "DS1073-01-2x1-MVT6"
+		(property "Product Name" "DS1073-01-2x1MR2T6"
 			(at 184.15 99.06 0)
 			(hide yes)
@@
 			)
 		)
-		(property "Description P/N" ""
+		(property "Description P/N" "Resistor SMD"
 			(at 128.27 109.22 0)
 			(hide yes)
@@
 			)
 		)
-		(property "Description P/N" ""
+		(property "Description P/N" "Capacitor SMD 50V"
 			(at 134.62 109.22 0)
 			(hide yes)
@@
 			)
 		)
-		(property "Value" "MF-SM075/60-2"
+		(property "Value" ""
 			(at 163.83 91.44 0)
 			(hide yes)
@@
 			(at 163.83 93.98 0)
 			(hide yes)
+			(show_name no)
+			(do_not_autoplace no)
+			(effects
+				(font
+					(size 1.27 1.27)
+				)
+			)
+		)
+		(property "Product Name" "MF-SM075/60-2"
+			(at 163.83 93.98 0)
+			(hide yes)
+			(show_name no)
+			(do_not_autoplace no)
+			(effects
+				(font
+					(size 1.27 1.27)
+				)
+			)
+		)
+		(property "Description P/N" "Fuse SMD"
+			(at 163.83 93.98 0)
+			(hide yes)
