File: Sch/Solenoid_control.kicad_sch (KiCad schematic)
At the start: 13 parts

Commit message: VER1.0: обновил шелкографию, гербера и BOM
Parts:
- R108, R109, R110, R120: Description P/N Resistor SMD -> Resistor SMD 1%
Changed lines of the file:
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@@
 			)
 		)
-		(property "Description P/N" "Resistor SMD"
+		(property "Description P/N" "Resistor SMD 1%"
 			(at 166.37 106.68 0)
 			(hide yes)
@@
 			)
 		)
-		(property "Description P/N" "Resistor SMD"
+		(property "Description P/N" "Resistor SMD 1%"
 			(at 137.16 96.52 0)
 			(hide yes)
@@
 			)
 		)
-		(property "Description P/N" "Resistor SMD"
+		(property "Description P/N" "Resistor SMD 1%"
 			(at 124.46 105.41 0)
 			(hide yes)
@@
 			)
 		)
-		(property "Description P/N" "Resistor SMD"
+		(property "Description P/N" "Resistor SMD 1%"
 			(at 128.27 109.22 0)
 			(hide yes)
