File: Sch/Flow_measure.kicad_sch (KiCad schematic)
At the start: 26 parts

Commit message: VER1.0: исправил каналы расходомеров, добавил папку с отчетным КД
Parts:
- removed J28: (no value), Connector_Molex:Molex_Mini-Fit_Jr_5569-02A2_2x01_P4.20mm_Horizontal, symbol Connector_Generic:Conn_01x02
- added J7: (no value), Connector_Molex:Molex_Mini-Fit_Jr_5569-04A2_2x02_P4.20mm_Horizontal, symbol Connector_Generic:Conn_02x02_Odd_Even
- renumbered C18 to C87, C19 to C88, C17 to C89, C22 to C90, C23 to C91, C3 to C92, C16 to C93, C4 to C94, C10 to C95, D2 to D15, R3 to R62, R9 to R63, R7 to R64, R8 to R65, R11 to R66, R5 to R67, R21 to R68, R10 to R69, R79 to R85, TP9 to TP15, TP17 to TP23, TP25 to TP31, TP1 to TP7, U2 to U17, U6 to U18
Connections:
- net +24V: now also J7.1 (Pin_1)
- net GNDD: now also J7.3 (Pin_3), J7.4 (Pin_4)
- net at R62.1, R63.1, TP23.1: now also J7.2 (Pin_2)
- net P_measure_MCU renamed F_measure_MCU
